Commit message: load_motion ok v1

File: assets/urdf/a1_ig.urdf (robot description, URDF)
Before this commit: robot a1, 23 links, 22 joints
Links:
- link FL_calf: mass 0.166 -> 0.151; geometry collision box size=0.2 0.016 0.016; visual mesh filename=../meshes/calf.dae scale=1 1 1
- link FL_hip: mass 0.696 -> 0.595; geometry visual mesh filename=../meshes/hip.dae scale=1 1 1
- link FL_thigh: mass 1.013 -> 0.888; geometry collision box size=0.2 0.0245 0.034; visual mesh filename=../meshes/thigh.dae scale=1 1 1
- link FR_calf: mass 0.166 -> 0.151; geometry collision box size=0.2 0.016 0.016; visual mesh filename=../meshes/calf.dae scale=1 1 1
- link FR_hip: mass 0.696 -> 0.595; geometry visual mesh filename=../meshes/hip.dae scale=1 1 1
- link FR_thigh: mass 1.013 -> 0.888; geometry collision box size=0.2 0.0245 0.034; visual mesh filename=../meshes/thigh_mirror.dae scale=1 1 1
- link RL_calf: mass 0.166 -> 0.151; geometry collision box size=0.2 0.016 0.016; visual mesh filename=../meshes/calf.dae scale=1 1 1
- link RL_hip: mass 0.696 -> 0.595; geometry visual mesh filename=../meshes/hip.dae scale=1 1 1
- link RL_thigh: mass 1.013 -> 0.888; geometry collision box size=0.2 0.0245 0.034; visual mesh filename=../meshes/thigh.dae scale=1 1 1
- link RR_calf: mass 0.166 -> 0.151; geometry collision box size=0.2 0.016 0.016; visual mesh filename=../meshes/calf.dae scale=1 1 1
- link RR_hip: mass 0.696 -> 0.595; geometry visual mesh filename=../meshes/hip.dae scale=1 1 1
- link RR_thigh: mass 1.013 -> 0.888; geometry collision box size=0.2 0.0245 0.034; visual mesh filename=../meshes/thigh_mirror.dae scale=1 1 1
- link trunk: mass 4.713 -> 6.0; geometry collision box size=0.267 0.194 0.114; visual mesh filename=../meshes/trunk.dae scale=1 1 1
Joints:
- removed joint FL_calf_joint
- removed joint FL_foot_fixed
- removed joint FL_hip_fixed
- removed joint FL_hip_joint
- removed joint FL_thigh_joint
- removed joint FR_calf_joint
- removed joint FR_foot_fixed
- removed joint FR_hip_fixed
- removed joint FR_hip_joint
- removed joint FR_thigh_joint
- removed joint RL_calf_joint
- removed joint RL_foot_fixed
- removed joint RL_hip_fixed
- removed joint RL_hip_joint
- removed joint RL_thigh_joint
- removed joint RR_calf_joint
- removed joint RR_foot_fixed
- removed joint RR_hip_fixed
- removed joint RR_hip_joint
- removed joint RR_thigh_joint
- added joint leg0_FR_a_hip_joint: type revolute, parent trunk, child FR_hip, origin xyz=0.1805 -0.047 0 rpy=0 0 0, axis 1 0 0, limit lower=-0.8028 upper=0.8028 effort=33.5 velocity=21
- added joint leg0_FR_b_hip_fixed: type fixed, parent FR_hip, child FR_thigh_shoulder, origin xyz=0 -0.081 0 rpy=0 0 0
- added joint leg0_FR_c_thigh_joint: type revolute, parent FR_hip, child FR_thigh, origin xyz=0 -0.0838 0 rpy=0 0 0, axis 0 1 0, limit lower=-1.0471975512 upper=4.188 effort=33.5 velocity=21
- added joint leg0_FR_d_calf_joint: type revolute, parent FR_thigh, child FR_calf, origin xyz=0 0 -0.2 rpy=0 0 0, axis 0 1 0, limit lower=-2.69653369433 upper=-0.916297857297 effort=33.5 velocity=21
- added joint leg0_FR_e_foot_fixed: type fixed, parent FR_calf, child FR_foot, origin xyz=0 0 -0.2 rpy=0 0 0
- added joint leg1_FL_a_hip_joint: type revolute, parent trunk, child FL_hip, origin xyz=0.1805 0.047 0 rpy=0 0 0, axis 1 0 0, limit lower=-0.8028 upper=0.8028 effort=33.5 velocity=21
- added joint leg1_FL_b_hip_fixed: type fixed, parent FL_hip, child FL_thigh_shoulder, origin xyz=0 0.081 0 rpy=0 0 0
- added joint leg1_FL_c_thigh_joint: type revolute, parent FL_hip, child FL_thigh, origin xyz=0 0.0838 0 rpy=0 0 0, axis 0 1 0, limit lower=-1.0471975512 upper=4.188 effort=33.5 velocity=21
- added joint leg1_FL_d_calf_joint: type revolute, parent FL_thigh, child FL_calf, origin xyz=0 0 -0.2 rpy=0 0 0, axis 0 1 0, limit lower=-2.69653369433 upper=-0.916297857297 effort=33.5 velocity=21
- added joint leg1_FL_e_foot_fixed: type fixed, parent FL_calf, child FL_foot, origin xyz=0 0 -0.2 rpy=0 0 0
- added joint leg2_RR_a_hip_joint: type revolute, parent trunk, child RR_hip, origin xyz=-0.1805 -0.047 0 rpy=0 0 0, axis 1 0 0, limit lower=-0.8028 upper=0.8028 effort=33.5 velocity=21
- added joint leg2_RR_b_hip_fixed: type fixed, parent RR_hip, child RR_thigh_shoulder, origin xyz=0 -0.081 0 rpy=0 0 0
- added joint leg2_RR_c_thigh_joint: type revolute, parent RR_hip, child RR_thigh, origin xyz=0 -0.0838 0 rpy=0 0 0, axis 0 1 0, limit lower=-1.0471975512 upper=4.188 effort=33.5 velocity=21
- added joint leg2_RR_d_calf_joint: type revolute, parent RR_thigh, child RR_calf, origin xyz=0 0 -0.2 rpy=0 0 0, axis 0 1 0, limit lower=-2.69653369433 upper=-0.916297857297 effort=33.5 velocity=21
- added joint leg2_RR_e_foot_fixed: type fixed, parent RR_calf, child RR_foot, origin xyz=0 0 -0.2 rpy=0 0 0
- added joint leg3_RL_a_hip_joint: type revolute, parent trunk, child RL_hip, origin xyz=-0.1805 0.047 0 rpy=0 0 0, axis 1 0 0, limit lower=-0.8028 upper=0.8028 effort=33.5 velocity=21
- added joint leg3_RL_b_hip_fixed: type fixed, parent RL_hip, child RL_thigh_shoulder, origin xyz=0 0.081 0 rpy=0 0 0
- added joint leg3_RL_c_thigh_joint: type revolute, parent RL_hip, child RL_thigh, origin xyz=0 0.0838 0 rpy=0 0 0, axis 0 1 0, limit lower=-1.0471975512 upper=4.188 effort=33.5 velocity=21
- added joint leg3_RL_d_calf_joint: type revolute, parent RL_thigh, child RL_calf, origin xyz=0 0 -0.2 rpy=0 0 0, axis 0 1 0, limit lower=-2.69653369433 upper=-0.916297857297 effort=33.5 velocity=21
- added joint leg3_RL_e_foot_fixed: type fixed, parent RL_calf, child RL_foot, origin xyz=0 0 -0.2 rpy=0 0 0

File: assets/urdf/a1_original.urdf (robot description, URDF)
Before this commit: robot a1_description, 23 links, 22 joints
Links:
- link FL_calf: geometry collision box size=0.2 0.016 0.016; visual mesh filename=../meshes/calf.dae scale=1 1 1
- link FL_hip: geometry visual mesh filename=../meshes/hip.dae scale=1 1 1
- link FL_thigh: geometry collision box size=0.2 0.0245 0.034; visual mesh filename=../meshes/thigh.dae scale=1 1 1
- link FR_calf: geometry collision box size=0.2 0.016 0.016; visual mesh filename=../meshes/calf.dae scale=1 1 1
- link FR_hip: geometry visual mesh filename=../meshes/hip.dae scale=1 1 1
- link FR_thigh: geometry collision box size=0.2 0.0245 0.034; visual mesh filename=../meshes/thigh_mirror.dae scale=1 1 1
- link RL_calf: geometry collision box size=0.2 0.016 0.016; visual mesh filename=../meshes/calf.dae scale=1 1 1
- link RL_hip: geometry visual mesh filename=../meshes/hip.dae scale=1 1 1
- link RL_thigh: geometry collision box size=0.2 0.0245 0.034; visual mesh filename=../meshes/thigh.dae scale=1 1 1
- link RR_calf: geometry collision box size=0.2 0.016 0.016; visual mesh filename=../meshes/calf.dae scale=1 1 1
- link RR_hip: geometry visual mesh filename=../meshes/hip.dae scale=1 1 1
- link RR_thigh: geometry collision box size=0.2 0.0245 0.034; visual mesh filename=../meshes/thigh_mirror.dae scale=1 1 1
- link trunk: geometry collision box size=0.267 0.194 0.114; visual mesh filename=../meshes/trunk.dae scale=1 1 1
