Commit message: go1_ig urdf

File: assets/urdf/a1_ig copy.urdf (robot description, URDF)
Before this commit: robot a1_description, 23 links, 22 joints
Links:
- link FL_calf: mass 0.131 -> 0.151; geometry collision box size=0.2 0.016 0.016; visual mesh filename=../meshes/calf.dae scale=1 1 1
- link FL_hip: mass 0.591 -> 0.595; geometry visual mesh filename=../meshes/hip.dae scale=1 1 1
- link FL_thigh: mass 0.92 -> 0.888; geometry collision box size=0.2 0.0245 0.034; visual mesh filename=../meshes/thigh.dae scale=1 1 1
- link FR_calf: mass 0.131 -> 0.151; geometry collision box size=0.2 0.016 0.016; visual mesh filename=../meshes/calf.dae scale=1 1 1
- link FR_hip: mass 0.591 -> 0.595; geometry visual mesh filename=../meshes/hip.dae scale=1 1 1
- link FR_thigh: mass 0.92 -> 0.888; geometry collision box size=0.2 0.0245 0.034; visual mesh filename=../meshes/thigh_mirror.dae scale=1 1 1
- link RL_calf: mass 0.131 -> 0.151; geometry collision box size=0.2 0.016 0.016; visual mesh filename=../meshes/calf.dae scale=1 1 1
- link RL_hip: mass 0.591 -> 0.595; geometry visual mesh filename=../meshes/hip.dae scale=1 1 1
- link RL_thigh: mass 0.92 -> 0.888; geometry collision box size=0.2 0.0245 0.034; visual mesh filename=../meshes/thigh.dae scale=1 1 1
- link RR_calf: mass 0.131 -> 0.151; geometry collision box size=0.2 0.016 0.016; visual mesh filename=../meshes/calf.dae scale=1 1 1
- link RR_hip: mass 0.591 -> 0.595; geometry visual mesh filename=../meshes/hip.dae scale=1 1 1
- link RR_thigh: mass 0.92 -> 0.888; geometry collision box size=0.2 0.0245 0.034; visual mesh filename=../meshes/thigh_mirror.dae scale=1 1 1
- link trunk: mass 5.204 -> 6.0; geometry collision box size=0.267 0.194 0.114; visual mesh filename=../meshes/trunk.dae scale=1 1 1
Joints:
- joint leg0_FR_a_hip_joint: limit lower=-1.0471975512 upper=1.0471975512 effort=23.7 velocity=30.1 -> lower=-0.8028 upper=0.8028 effort=33.5 velocity=21; origin xyz=0.1881 -0.04675 0 rpy=0 0 0 -> xyz=0.1805 -0.047 0 rpy=0 0 0
- joint leg0_FR_c_thigh_joint: limit lower=-0.663225115758 upper=2.96705972839 effort=23.7 velocity=30.1 -> lower=-1.0471975512 upper=4.188 effort=33.5 velocity=21; origin xyz=0 -0.08 0 rpy=0 0 0 -> xyz=0 -0.0838 0 rpy=0 0 0
- joint leg0_FR_d_calf_joint: limit lower=-2.72271363311 upper=-0.837758040957 effort=23.7 velocity=30.1 -> lower=-2.69653369433 upper=-0.916297857297 effort=33.5 velocity=21; origin xyz=0 0 -0.213 rpy=0 0 0 -> xyz=0 0 -0.2 rpy=0 0 0
- joint leg0_FR_e_foot_fixed: origin xyz=0 0 -0.213 rpy=0 0 0 -> xyz=0 0 -0.2 rpy=0 0 0
- joint leg1_FL_a_hip_joint: limit lower=-1.0471975512 upper=1.0471975512 effort=23.7 velocity=30.1 -> lower=-0.8028 upper=0.8028 effort=33.5 velocity=21; origin xyz=0.1881 0.04675 0 rpy=0 0 0 -> xyz=0.1805 0.047 0 rpy=0 0 0
- joint leg1_FL_c_thigh_joint: limit lower=-0.663225115758 upper=2.96705972839 effort=23.7 velocity=30.1 -> lower=-1.0471975512 upper=4.188 effort=33.5 velocity=21; origin xyz=0 0.08 0 rpy=0 0 0 -> xyz=0 0.0838 0 rpy=0 0 0
- joint leg1_FL_d_calf_joint: limit lower=-2.72271363311 upper=-0.837758040957 effort=23.7 velocity=30.1 -> lower=-2.69653369433 upper=-0.916297857297 effort=33.5 velocity=21; origin xyz=0 0 -0.213 rpy=0 0 0 -> xyz=0 0 -0.2 rpy=0 0 0
- joint leg1_FL_e_foot_fixed: origin xyz=0 0 -0.213 rpy=0 0 0 -> xyz=0 0 -0.2 rpy=0 0 0
- joint leg2_RR_a_hip_joint: limit lower=-1.0471975512 upper=1.0471975512 effort=23.7 velocity=30.1 -> lower=-0.8028 upper=0.8028 effort=33.5 velocity=21; origin xyz=-0.1881 -0.04675 0 rpy=0 0 0 -> xyz=-0.1805 -0.047 0 rpy=0 0 0
- joint leg2_RR_c_thigh_joint: limit lower=-0.663225115758 upper=2.96705972839 effort=23.7 velocity=30.1 -> lower=-1.0471975512 upper=4.188 effort=33.5 velocity=21; origin xyz=0 -0.08 0 rpy=0 0 0 -> xyz=0 -0.0838 0 rpy=0 0 0
- joint leg2_RR_d_calf_joint: limit lower=-2.72271363311 upper=-0.837758040957 effort=23.7 velocity=30.1 -> lower=-2.69653369433 upper=-0.916297857297 effort=33.5 velocity=21; origin xyz=0 0 -0.213 rpy=0 0 0 -> xyz=0 0 -0.2 rpy=0 0 0
- joint leg2_RR_e_foot_fixed: origin xyz=0 0 -0.213 rpy=0 0 0 -> xyz=0 0 -0.2 rpy=0 0 0
- joint leg3_RL_a_hip_joint: limit lower=-1.0471975512 upper=1.0471975512 effort=23.7 velocity=30.1 -> lower=-0.8028 upper=0.8028 effort=33.5 velocity=21; origin xyz=-0.1881 0.04675 0 rpy=0 0 0 -> xyz=-0.1805 0.047 0 rpy=0 0 0
- joint leg3_RL_c_thigh_joint: limit lower=-0.663225115758 upper=2.96705972839 effort=23.7 velocity=30.1 -> lower=-1.0471975512 upper=4.188 effort=33.5 velocity=21; origin xyz=0 0.08 0 rpy=0 0 0 -> xyz=0 0.0838 0 rpy=0 0 0
- joint leg3_RL_d_calf_joint: limit lower=-2.72271363311 upper=-0.837758040957 effort=23.7 velocity=30.1 -> lower=-2.69653369433 upper=-0.916297857297 effort=33.5 velocity=21; origin xyz=0 0 -0.213 rpy=0 0 0 -> xyz=0 0 -0.2 rpy=0 0 0
- joint leg3_RL_e_foot_fixed: origin xyz=0 0 -0.213 rpy=0 0 0 -> xyz=0 0 -0.2 rpy=0 0 0
